File: rfidsecuritysystemV2/rfidsecuritysystemV2.kicad_pcb (KiCad board)
At the start: 2 copper layers, 25.4 x 63.5 mm, 15 parts, among them J2 Conn_01x06_Socket, J3 Conn_01x02_Socket, J4 Conn_01x02_Socket, J5 Conn_01x20_Socket, J6 Conn_01x20_Socket, SW1 SW_Push

Commit message: finish v2
Connections:
- BZ1 pad 1: Net-(BZ1--) -> /GPIO 22
- BZ1 pad 2: Net-(BZ1-+) -> GND
- D1 pad 1: Net-(BZ1-+) -> GND
- D2 pad 1: Net-(BZ1-+) -> GND
- J2 pad 1: Net-(J1-Pin_2) -> +5V
- J2 pad 2: Net-(BZ1-+) -> GND
- J2 pad 4: Net-(J1-Pin_8) -> /UART TX
- J2 pad 5: Net-(J1-Pin_10) -> /UART RX
- J3 pad 1: Net-(BZ1-+) -> GND
- J3 pad 2: Net-(J1-Pin_22) -> /GPIO 21
- J4 pad 1: Net-(J1-Pin_25) -> /GPIO 16
- J4 pad 2: Net-(BZ1-+) -> GND
- J5 pad 14: unconnected-(J5-Pin_14-Pad14) -> /GPIO 10
- J5 pad 16: unconnected-(J5-Pin_16-Pad16) -> /UART TX
- J5 pad 17: unconnected-(J5-Pin_17-Pad17) -> /UART RX
- J5 pad 7: unconnected-(J5-Pin_7-Pad7) -> /GPIO 5
- J5 pad 9: unconnected-(J5-Pin_9-Pad9) -> /GPIO 6
- J6 pad 12: unconnected-(J6-Pin_12-Pad12) -> /GPIO 22
- J6 pad 14: unconnected-(J6-Pin_14-Pad14) -> /GPIO 21
- J6 pad 2: unconnected-(J6-Pin_2-Pad2) -> +5V
- J6 pad 20: unconnected-(J6-Pin_20-Pad20) -> /GPIO 16
- J6 pad 3: unconnected-(J6-Pin_3-Pad3) -> GND
- R1 pad 2: Net-(J1-Pin_24) -> /GPIO 6
- R2 pad 2: Net-(J1-Pin_17) -> /GPIO 5
- SW1 pad 1: Net-(BZ1-+) -> GND
- SW1 pad 2: Net-(J1-Pin_23) -> /GPIO 10
Routing:
- net GND: track 0.00 -> 71.0 mm
- net Net-(BZ1-+): track 58.0 -> 0.00 mm
- net +5V: track 0.00 -> 39.0 mm
- net /GPIO 22: track 0.00 -> 23.7 mm
- net /GPIO 10: track 0.00 -> 12.8 mm
- net /UART TX: track 0.00 -> 8.98 mm
- net /GPIO 21: track 0.00 -> 8.98 mm
- net /UART RX: track 0.00 -> 8.98 mm
- net /GPIO 16: track 0.00 -> 7.93 mm
- net Net-(J1-Pin_23): track 6.50 -> 0.00 mm
- net /GPIO 6: track 0.00 -> 4.34 mm
- net /GPIO 5: track 0.00 -> 4.34 mm
Other:
- board text added: "© Anders P 1/22/2024 Raspberry Pi RFID Security System"
- board text removed: "© Anders P 7/5/2023 Raspberry Pi RFID Security System"
