File: rfidsecuritysystemV2/rfidsecuritysystemV2.kicad_sch (KiCad schematic)
At the start: 17 parts, among them J1 Conn_02x20_Odd_Even, J2 Conn_01x06_Socket, J3 Conn_01x02_Socket, J4 Conn_01x02_Socket, J5 Conn_01x20_Socket, J6 Conn_01x20_Socket, SW1 SW_Push, U1 Pico

Commit message: finish v2
Connections:
- net GPIO 6: now reaches J1.24 (Pin_24), R1.2
- net GPIO 6: now also J5.9 (Pin_9)
- net +5V: now reaches J1.2 (Pin_2), J2.1 (Pin_1)
- net +5V: now also J6.2 (Pin_2)
- net GND: now reaches BZ1.2 (+), D1.1 (K), D2.1 (K), J1.6 (Pin_6), J2.2 (Pin_2), J3.1 (Pin_1), J4.2 (Pin_2), SW1.1
- net GND: now also J6.3 (Pin_3)
- net UART TX: now reaches J1.8 (Pin_8), J2.4 (Pin_4)
- net UART TX: now also J5.16 (Pin_16)
- net UART RX: now reaches J1.10 (Pin_10), J2.5 (Pin_5)
- net UART RX: now also J5.17 (Pin_17)
- net GPIO 10: now reaches J5.14 (Pin_14)
- net GPIO 10: now also J1.23 (Pin_23), SW1.2
- net GPIO 5: now reaches J5.7 (Pin_7)
- net GPIO 5: now also J1.17 (Pin_17), R2.2
- net GPIO 22: now reaches BZ1.1 (-), J1.27 (Pin_27)
- net GPIO 22: now also J6.12 (Pin_12)
- net GPIO 21: now reaches J6.14 (Pin_14)
- net GPIO 21: now also J1.22 (Pin_22), J3.2 (Pin_2)
- net GPIO 16: now reaches J6.20 (Pin_20)
- net GPIO 16: now also J1.31 (Pin_31), J4.1 (Pin_1)
- net at J1.25 (Pin_25): no longer J4.1 (Pin_1)
Other:
- moved on the sheet: J5, J6
